Commit message: A gripper was added to the arm-only version of Aloha

File: src/curobo/content/assets/robot/aloha/aloha_v1_1arm.urdf (robot description, URDF)
Before this commit: robot bimanual_viperx_transfer_cube, 9 links, 8 joints
Links:
- removed link tool0
- added link vx300s_left_gripper_prop_link, mass 0.008009; collision mesh filename=meshes/vx300s_8_gripper_prop.stl scale=0.001 0.001 0.001; visual mesh filename=meshes/vx300s_8_gripper_prop.stl scale=0.001 0.001 0.001
- added link vx300s_left_left_finger_link, mass 0.0348; collision mesh filename=meshes/vx300s_10_custom_finger_left.stl scale=0.001 0.001 0.001; visual mesh filename=meshes/vx300s_10_custom_finger_left.stl scale=0.001 0.001 0.001
- added link vx300s_left_right_finger_link, mass 0.0348; collision mesh filename=meshes/vx300s_10_custom_finger_right.stl scale=0.001 0.001 0.001; visual mesh filename=meshes/vx300s_10_custom_finger_right.stl scale=0.001 0.001 0.001
Joints:
- added joint vx300s_left_left_finger: type prismatic, parent vx300s_left_gripper_link, child vx300s_left_left_finger_link, origin xyz=0.0737 -0.031 0 rpy=0 1.57 0, axis 0 1 0, limit lower=0.0 upper=0.0605 effort=100 velocity=1.0
- added joint vx300s_left_right_finger: type prismatic, parent vx300s_left_gripper_link, child vx300s_left_right_finger_link, origin xyz=0.0737 0.031 0.0 rpy=0 1.57 0, axis 0 1 0, limit lower=-0.0605 upper=-0.0 effort=100 velocity=1.0, mimic joint=vx300s_left_left_finger multiplier=-1.0 offset=0.0
- joint vx300s_left_gripper: child tool0 -> vx300s_left_gripper_prop_link
